File: Sound Defense Proto Board/SD_ProtoBoard/SD_ProtoBoard.kicad_sch (KiCad schematic)
At the start: 14 parts, among them IC1 ATTINY402-SSNR, IC2 PAM8906M1018-13, J1 TD-104-T-A, J2 WJ500V-5.08-2P, U1 3025 3v Battery Holder

Commit message: New DEV Board and Code
Parts:
- removed J1: TD-104-T-A, SD-HEAD:SAMTEC_TD-104-T-A, symbol Symbols:TD-104-T-A
- removed J2: WJ500V-5.08-2P, SD-SCR-TERM:WJ500V5082P, symbol Symbols:WJ500V-5.08-2P
- removed U1: 3025 3v Battery Holder, SD-BAT-HOL:3025, symbol Symbols:3025
- added C6, C7: 10uF GRM188R61E106MA73D, SD-CAP-10:CAPC1608X90N, symbol Symbols:GRM188R61E106MA73D
- added IC3: MCP73831T-2ACI_OT, SD-MCP:SOT95P270X145-5N, symbol SD_LIB:MCP73831T-2ACI_OT
- added J1: Conn_01x03_Pin, Connector_PinHeader_2.54mm:PinHeader_1x03_P2.54mm_Vertical, symbol Connector:Conn_01x03_Pin
- added J3: USB_C_Receptacle_PowerOnly_6P, Connector_USB:USB_C_Receptacle_GCT_USB4125-xx-x-0190_6P_TopMnt_Horizontal, symbol Connector:USB_C_Receptacle_PowerOnly_6P
- added J4: S2B-PH-SM4-TB_LF__SN_, SD-JST3:S2BPHSM4TBLFSN, symbol SD_LIB:S2B-PH-SM4-TB_LF__SN_
- added R1, R3: 5.1KOhm, SD-RES-5_1K:RESC1005X40N, symbol SD_LIB:0402WGF5101TCE
- added R4: 10K Ohm, SD-RES-10K:RESC1005X40N, symbol SD_LIB:0402WGF1002TCE
- added X1: CPT-1404-85T, SD-PIEZO:SD-CPT-1404-85T, symbol SD_LIB:CPT-1404-85T
- R2: value RC0402FR-07100RL -> 100 Ohms
Connections:
- net GND: now also LED1.2 (A), C6.1, C7.2, IC3.2 (VSS), J1.2 (Pin_2), J3.A12 (GND), J3.B12 (GND), J4.1, R1.1, R3.1, R4.2; no longer LED1.1 (K)
- net at R2.1: now also LED1.1 (K); no longer IC1.7 (PA3/EXTCLK)
- net UPDI: now reaches IC1.6 (PA0/~{RESET}/UPDI)
- net UPDI: now also J1.3 (Pin_3)
- net at R2.2: now also IC3.1 (STAT); no longer LED1.2 (A)
- net at IC2.6 (OUTN): now also X1.2
- net at IC2.7 (OUTP): now also X1.1
- net VCC renamed VBAT
- net VBAT: now also C7.1, IC3.3 (VBAT), J1.1 (Pin_1), J4.2
- new net: IC3.5 (PROG), R4.1
- new net: C6.2, IC3.4 (VDD), J3.A9 (VBUS), J3.B9 (VBUS)
- new net: J3.B5 (CC2), R3.2
- new net: J3.A5 (CC1), R1.2
- no-connect marks 2 -> 8
Other:
- moved on the sheet: C1, C2, C3, C4, C5, IC1, IC2, L1, LED1, R2, S1

Commit message: Production Board v1-0
Parts:
- removed J1: Conn_01x03_Pin, Connector_PinHeader_2.54mm:PinHeader_1x03_P2.54mm_Vertical, symbol Connector:Conn_01x03_Pin
- removed J3: USB_C_Receptacle_PowerOnly_6P, Connector_USB:USB_C_Receptacle_GCT_USB4125-xx-x-0190_6P_TopMnt_Horizontal, symbol Connector:USB_C_Receptacle_PowerOnly_6P
- removed J4: S2B-PH-SM4-TB_LF__SN_, SD-JST3:S2BPHSM4TBLFSN, symbol SD_LIB:S2B-PH-SM4-TB_LF__SN_
- removed X1: CPT-1404-85T, SD-PIEZO:SD-CPT-1404-85T, symbol SD_LIB:CPT-1404-85T
- added H1, H3: MountingHole, MountingHole:MountingHole_2.2mm_M2, symbol Mechanical:MountingHole
- added J1: MC-306LS-H50, SD-USB-C-SHORT:MC-306LS-H50, symbol SD_LIB:USB-C_TOP
- added LS1: CPT-1762-90-SMT-TR, SD-SMD-BUZZER:XDCR_CPT-1762-90-SMT-TR, symbol SD_LIB:CPT-1762-90-SMT-TR
- added TP1: UPDI, TestPoint:TestPoint_Pad_2.5x2.5mm, symbol Connector:TestPoint
- added TP2: VCC, TestPoint:TestPoint_Pad_2.5x2.5mm, symbol Connector:TestPoint
- added TP3: GND, TestPoint:TestPoint_Pad_3.0x3.0mm, symbol Connector:TestPoint
- added U1: LP402025, Battery:LP402025, symbol Battery_Management:LP402025
- C1: value 0.1uF 0402B104K160CT -> 0.1uF
- C2, C4, C5: value 1uF GRM155R61E105KA12D -> 1uF; footprint SD-CAP1:CAPC1005X55N -> SD-01-CAP:CAPC1005X55N
- C3, C6, C7: value 10uF GRM188R61E106MA73D -> 10uF
- L1: footprint SD-IND:INDC2016X95N -> SD-INDUCTOR:INDC2016X95N
- LED1: value 150060VS75000 -> CHARGE INDICATOR
- R1, R3: value 5.1KOhm -> 5.1K
- R4: value 10K Ohm -> 10K
- S1: value 436331045822 -> SIDE SWITCH
Connections:
- net GND: now also J1.A12 (GND), J1.B12 (GND), TP3.1, U1.2 (GND)
- net UPDI: now also TP1.1
- net VBAT: now also TP2.1, U1.1 (3.7V)
- net at IC2.6 (OUTN): now also LS1.N
- net at IC2.7 (OUTP): now also LS1.P
- net PWM: now reaches IC1.3 (PA7), IC2.9 (DIN)
- net at C6.2, IC3.4 (VDD): now also J1.A9 (VBUS), J1.B9 (VBUS)
- net BUTTON: now reaches IC1.5 (PA2), S1.2 (NO_1)
- net at R3.2: now also J1.A5 (CC1)
- net at R1.2: now also J1.B5 (CC2)
- no-connect marks 8 -> 7
Other:
- moved on the sheet: C1, C2, C3, C4, C5, C6, C7, IC1, IC2, IC3, L1, LED1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

Commit message: 4677-901 v2.0
Parts:
- removed H1, H3: MountingHole, MountingHole:MountingHole_2.2mm_M2, symbol Mechanical:MountingHole
- added LED2: TEST LED, LED:LEDC1608X80N, symbol SD_LIB:150060VS75000
- added R5: 100 Ohms, SD-RES:RESC1005X40N, symbol SD_LIB:RC0402FR-07100RL
Connections:
- net BUTTON is gone; now on net NO_1: IC1.5 (PA2), S1.2 (NO_1)
- net GND: now also C2.2, C6.2, J1.8, J1.9, LED1.1 (K), R1.2, R3.2, S1.3 (COM_2), LED2.1 (K); no longer C2.1, C6.1, LED1.2 (A), R1.1, R3.1
- net STAT: now reaches R2.1
- net STAT: now also IC3.1 (STAT); no longer LED1.1 (K)
- net at R2.2: now also LED1.2 (A); no longer IC3.1 (STAT)
- net at IC2.1 (VCC): now also C2.1; no longer C5.1
- net at IC2.5 (VOUT), IC2.8 (FB): now also C5.1; no longer C2.2
- net at IC3.4 (VDD), J1.A9 (VBUS), J1.B9 (VBUS): now also C6.1; no longer C6.2
- net TEST: now reaches IC1.7 (PA3/EXTCLK)
- net TEST: now also R5.1
- net NO_1: now reaches S1.4 (NO_2)
- net CC1: now reaches J1.A5 (CC1)
- net CC1: now also R3.1; no longer R3.2
- net CC2: now reaches J1.B5 (CC2)
- net CC2: now also R1.1; no longer R1.2
- net VBAT renamed VCC
- new net: LED2.2 (A), R5.2
- no-connect marks 7 -> 2
Other:
- title: Sound Defense Dev Board -> Sound Defense Production PCB
- moved on the sheet: C1, C2, C3, C4, C5, C6, C7, IC1, IC2, IC3, J1, L1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

Commit message: New
Parts:
- removed LED1: CHARGE INDICATOR, LED:LEDC1608X80N, symbol SD_LIB:150060VS75000
- removed R2: 100 Ohms, SD-RES:RESC1005X40N, symbol SD_LIB:RC0402FR-07100RL
- added LED1: 18-225A/R6GHC-A01/3T, 4677-Footprints:18-225A R6GHC-A01 3T, symbol 4677-Library:18-225A/R6GHC-A01/3T
- added R2, R6: 100 Ohms, 4677-Footprints:RESC1005X40N, symbol 4677-Library:RC0402FR-07100RL
- C1: footprint SD-01-CAP:CAPC1005X55N -> 4677-Footprints:CAPC1005X55N; symbol Symbols:0402B104K160CT -> 4677-Library:0402B104K160CT
- C2, C4, C5: footprint SD-01-CAP:CAPC1005X55N -> 4677-Footprints:CAPC1005X55N; symbol Symbols:GRM155R61E105KA12D -> 4677-Library:GRM155R61E105KA12D
- C3, C6, C7: footprint SD-CAP-10:CAPC1608X90N -> 4677-Footprints:CAPC1608X90N; symbol Symbols:GRM188R61E106MA73D -> 4677-Library:GRM188R61E106MA73D
- IC1: footprint SD-ATTINY:SOIC127P600X175-8N -> 4677-Footprints:SOIC127P600X175-8N; symbol Symbols:ATTINY402-SSNR -> 4677-Library:ATTINY402-SSNR
- IC2: footprint SD-PAM:SOP50P490X110-10N -> 4677-Footprints:SOP50P490X110-10N; symbol Symbols:PAM8906M1018-13 -> 4677-Library:PAM8906M1018-13
- IC3: footprint SD-MCP:SOT95P270X145-5N -> 4677-Footprints:SOT95P270X145-5N; symbol SD_LIB:MCP73831T-2ACI_OT -> 4677-Library:MCP73831T-2ACI_OT
- J1: footprint SD-USB-C-SHORT:MC-306LS-H50 -> 4677-Footprints:MC-306LS-H50; symbol SD_LIB:USB-C_TOP -> 4677-Library:USB-C_TOP
- L1: footprint SD-INDUCTOR:INDC2016X95N -> 4677-Footprints:INDC2016X95N; symbol Symbols:SRN2009T-R47M -> 4677-Library:SRN2009T-R47M
- LED2: footprint LED:LEDC1608X80N -> 4677-Footprints:LEDC1608X80N; symbol SD_LIB:150060VS75000 -> 4677-Library:150060VS75000
- LS1: footprint SD-SMD-BUZZER:XDCR_CPT-1762-90-SMT-TR -> 4677-Footprints:XDCR_CPT-1762-90-SMT-TR; symbol SD_LIB:CPT-1762-90-SMT-TR -> 4677-Library:CPT-1762-90-SMT-TR
- R1, R3: footprint SD-RES-5_1K:RESC1005X40N -> 4677-Footprints:RESC1005X40N; symbol SD_LIB:0402WGF5101TCE -> 4677-Library:0402WGF5101TCE
- R4: footprint SD-RES-10K:RESC1005X40N -> 4677-Footprints:RESC1005X40N; symbol SD_LIB:0402WGF1002TCE -> 4677-Library:0402WGF1002TCE
- R5: footprint SD-RES:RESC1005X40N -> 4677-Footprints:RESC1005X40N; symbol SD_LIB:RC0402FR-07100RL -> 4677-Library:RC0402FR-07100RL
- S1: footprint SD-SWI:436331045822 -> 4677-Footprints:436331045822; symbol Symbols:436331045822 -> 4677-Library:436331045822
- TP1, TP2: footprint TestPoint:TestPoint_Pad_2.5x2.5mm -> 4677-Footprints:TestPoint_Pad_2.5x2.5mm; symbol Connector:TestPoint -> 4677-Library:TestPoint
- TP3: footprint TestPoint:TestPoint_Pad_3.0x3.0mm -> 4677-Footprints:TestPoint_Pad_3.0x3.0mm; symbol Connector:TestPoint -> 4677-Library:TestPoint
- U1: value LP402025 -> Molex: 781710002; footprint Battery:LP402025 -> 4677-Footprints:CONN02_781710002_MOL; symbol Battery_Management:LP402025 -> 4677-Library:LP402025
Connections:
- net GND: now also LED1.4 (K2)
- net STAT: now also R2.1, R6.1
- net VDD: now reaches C6.1, IC3.4 (VDD), J1.A9 (VBUS), J1.B9 (VBUS)
- net VDD: now also LED1.2 (A1)
- new net: LED1.3 (K1), R6.2
- new net: LED1.1 (A2), R2.2
